File: work/pll-schematic/pll-schematic.kicad_sch (KiCad schematic)
At the start: 9 parts, among them U1 4046, U2 74LS163, U3 74LS163

Commit message: add output, whoops
Parts:
- added C1: 1n, symbol Device:C
- gave numbers to parts that had none: 2
- renumbered C1 to C2, C2 to C3, C3 to C5, R1 to R2
Connections:
- net at U1.4 (FOUT), U2.2 (CP), U3.2 (CP): now also C1.2
- new net freq. out: C1.1
Changed lines of the file:
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@@
   (junction (at 219.71 93.98) (diameter 0) (color 0 0 0 0)
+  )
+  (junction (at 73.66 82.55) (diameter 0) (color 0 0 0 0)
   )
   (junction (at 106.68 114.3) (diameter 0) (color 0 0 0 0)
@@
     (stroke (width 0) (type default) (color 0 0 0 0))
   )
+  (wire (pts (xy 73.66 82.55) (xy 73.66 129.54))
+    (stroke (width 0) (type default) (color 0 0 0 0))
+  )
   (wire (pts (xy 100.33 60.96) (xy 100.33 66.04))
     (stroke (width 0) (type default) (color 0 0 0 0))
@@
     (stroke (width 0) (type default) (color 0 0 0 0))
   )
+  (wire (pts (xy 67.31 82.55) (xy 73.66 82.55))
+    (stroke (width 0) (type default) (color 0 0 0 0))
+  )
   (wire (pts (xy 102.87 91.44) (xy 102.87 95.25))
     (stroke (width 0) (type default) (color 0 0 0 0))
@@
     (stroke (width 0) (type default) (color 0 0 0 0))
   )
-  (wire (pts (xy 73.66 129.54) (xy 73.66 60.96))
+  (wire (pts (xy 73.66 60.96) (xy 73.66 82.55))
     (stroke (width 0) (type default) (color 0 0 0 0))
   )
@@
   (wire (pts (xy 95.25 91.44) (xy 97.79 91.44))
     (stroke (width 0) (type default) (color 0 0 0 0))
+  )
+  (global_label "freq. out" (shape output) (at 59.69 82.55 180) (fields_autoplaced)
+    (effects (font (size 1.27 1.27)) (justify right))
+    (property "Intersheet References" "${INTERSHEET_REFS}" (id 0) (at 48.9312 82.4706 0)
+      (effects (font (size 1.27 1.27)) (justify right) hide)
+    )
   )
   (global_label "from teensy" (shape input) (at 59.69 96.52 180) (fields_autoplaced)
@@
   (symbol (lib_id "Device:C") (at 109.22 107.95 0) (unit 1)
     (in_bom yes) (on_board yes) (fields_autoplaced)
-    (property "Reference" "C3" (id 0) (at 113.03 106.6799 0)
+    (property "Reference" "C5" (id 0) (at 113.03 106.6799 0)
       (effects (font (size 1.27 1.27)) (justify left))
     )
@@
   (symbol (lib_id "power:GND") (at 240.03 83.82 0) (unit 1)
     (in_bom yes) (on_board yes) (fields_autoplaced)
-    (property "Reference" "#PWR08" (id 0) (at 240.03 90.17 0)
+    (property "Reference" "#PWR09" (id 0) (at 240.03 90.17 0)
       (effects (font (size 1.27 1.27)) hide)
     )
@@
   (symbol (lib_id "Device:C") (at 63.5 96.52 90) (unit 1)
     (in_bom yes) (on_board yes) (fields_autoplaced)
-    (property "Reference" "C1" (id 0) (at 63.5 88.9 90))
+    (property "Reference" "C2" (id 0) (at 63.5 88.9 90))
     (property "Value" "1n" (id 1) (at 63.5 91.44 90))
     (property "Footprint" "" (id 2) (at 67.31 95.5548 0)
@@
   (symbol (lib_id "power:VCC") (at 191.77 73.66 0) (unit 1)
     (in_bom yes) (on_board yes) (fields_autoplaced)
-    (property "Reference" "#PWR07" (id 0) (at 191.77 77.47 0)
+    (property "Reference" "#PWR08" (id 0) (at 191.77 77.47 0)
       (effects (font (size 1.27 1.27)) hide)
     )
@@
   (symbol (lib_id "power:GND") (at 179.07 83.82 0) (unit 1)
     (in_bom yes) (on_board yes) (fields_autoplaced)
-    (property "Reference" "#PWR06" (id 0) (at 179.07 90.17 0)
+    (property "Reference" "#PWR07" (id 0) (at 179.07 90.17 0)
       (effects (font (size 1.27 1.27)) hide)
     )
@@
   (symbol (lib_id "power:GND") (at 123.19 83.82 0) (unit 1)
     (in_bom yes) (on_board yes) (fields_autoplaced)
-    (property "Reference" "#PWR04" (id 0) (at 123.19 90.17 0)
+    (property "Reference" "#PWR05" (id 0) (at 123.19 90.17 0)
       (effects (font (size 1.27 1.27)) hide)
     )
@@
   (symbol (lib_id "Device:R_US") (at 104.14 107.95 0) (unit 1)
     (in_bom yes) (on_board yes)
-    (property "Reference" "R1" (id 0) (at 97.79 106.68 0)
+    (property "Reference" "R2" (id 0) (at 97.79 106.68 0)
       (effects (font (size 1.27 1.27)) (justify left))
     )
@@
   (symbol (lib_id "power:GND") (at 115.57 62.23 0) (unit 1)
     (in_bom yes) (on_board yes) (fields_autoplaced)
-    (property "Reference" "#PWR?" (id 0) (at 115.57 68.58 0)
+    (property "Reference" "#PWR04" (id 0) (at 115.57 68.58 0)
       (effects (font (size 1.27 1.27)) hide)
     )
@@
   (symbol (lib_id "Device:C") (at 99.06 95.25 90) (unit 1)
     (in_bom yes) (on_board yes)
-    (property "Reference" "C2" (id 0) (at 99.06 99.06 90))
+    (property "Reference" "C3" (id 0) (at 99.06 99.06 90))
     (property "Value" "47p" (id 1) (at 99.06 101.6 90))
     (property "Footprint" "" (id 2) (at 102.87 94.2848 0)
@@
   (symbol (lib_id "Device:R_US") (at 96.52 60.96 90) (unit 1)
     (in_bom yes) (on_board yes) (fields_autoplaced)
-    (property "Reference" "R?" (id 0) (at 96.52 54.61 90))
+    (property "Reference" "R1" (id 0) (at 96.52 54.61 90))
     (property "Value" "33k" (id 1) (at 96.52 57.15 90))
     (property "Footprint" "" (id 2) (at 96.774 59.944 90)
@@
   (symbol (lib_id "Device:C") (at 106.68 60.96 90) (unit 1)
     (in_bom yes) (on_board yes) (fields_autoplaced)
-    (property "Reference" "C?" (id 0) (at 106.68 53.34 90))
+    (property "Reference" "C4" (id 0) (at 106.68 53.34 90))
     (property "Value" "100p" (id 1) (at 106.68 55.88 90))
     (property "Footprint" "" (id 2) (at 110.49 59.9948 0)
@@
   (symbol (lib_id "power:VCC") (at 130.81 73.66 0) (unit 1)
     (in_bom yes) (on_board yes) (fields_autoplaced)
-    (property "Reference" "#PWR05" (id 0) (at 130.81 77.47 0)
+    (property "Reference" "#PWR06" (id 0) (at 130.81 77.47 0)
       (effects (font (size 1.27 1.27)) hide)
     )
@@
     )
     (pin "1")
+  )
+  (symbol (lib_id "Device:C") (at 63.5 82.55 90) (unit 1)
+    (in_bom yes) (on_board yes) (fields_autoplaced)
+    (property "Reference" "C1" (id 0) (at 63.5 74.93 90))
+    (property "Value" "1n" (id 1) (at 63.5 77.47 90))
+    (property "Footprint" "" (id 2) (at 67.31 81.5848 0)
+      (effects (font (size 1.27 1.27)) hide)
+    )
+    (property "Datasheet" "~" (id 3) (at 63.5 82.55 0)
+      (effects (font (size 1.27 1.27)) hide)
+    )
+    (pin "1")
+    (pin "2")
   )
   (symbol (lib_id "74xx:74LS163") (at 217.17 78.74 90) (unit 1)
@@
       (reference "#PWR03") (unit 1) (value "GND") (footprint "")
     )
+    (path "/792b677e-7f74-41d3-a77d-f64724e1ccbb"
+      (reference "#PWR04") (unit 1) (value "GND") (footprint "")
+    )
     (path "/68e1dd4b-4063-4612-8ead-c77420b7b652"
-      (reference "#PWR04") (unit 1) (value "GND") (footprint "")
+      (reference "#PWR05") (unit 1) (value "GND") (footprint "")
     )
     (path "/e574dd0d-e46f-40f8-b3e2-45c382ac9473"
-      (reference "#PWR05") (unit 1) (value "VCC") (footprint "")
+      (reference "#PWR06") (unit 1) (value "VCC") (footprint "")
     )
     (path "/566e953a-4572-4e6e-9f3f-b5d7c44820ca"
-      (reference "#PWR06") (unit 1) (value "GND") (footprint "")
+      (reference "#PWR07") (unit 1) (value "GND") (footprint "")
     )
     (path "/2a7b1f7e-8b3e-40dc-a41e-e958a80536aa"
-      (reference "#PWR07") (unit 1) (value "VCC") (footprint "")
+      (reference "#PWR08") (unit 1) (value "VCC") (footprint "")
     )
     (path "/15b53327-3530-4a1a-9580-2cfbd558ba27"
-      (reference "#PWR08") (unit 1) (value "GND") (footprint "")
-    )
-    (path "/792b677e-7f74-41d3-a77d-f64724e1ccbb"
-      (reference "#PWR?") (unit 1) (value "GND") (footprint "")
+      (reference "#PWR09") (unit 1) (value "GND") (footprint "")
+    )
+    (path "/eb9447ce-03f2-4cd9-a408-667a987bc7f7"
+      (reference "C1") (unit 1) (value "1n") (footprint "")
     )
     (path "/2846f4c9-5e76-48e4-8e8e-d1f6c65c6980"
-      (reference "C1") (unit 1) (value "1n") (footprint "")
+      (reference "C2") (unit 1) (value "1n") (footprint "")
     )
     (path "/c4cca214-064d-4db8-85cf-1491ad675840"
-      (reference "C2") (unit 1) (value "47p") (footprint "")
+      (reference "C3") (unit 1) (value "47p") (footprint "")
+    )
+    (path "/d7ceb106-986f-4792-af19-7e621a6094bb"
+      (reference "C4") (unit 1) (value "100p") (footprint "")
     )
     (path "/053c93ba-5464-4d78-ac2b-367e7ad9c633"
-      (reference "C3") (unit 1) (value "1n") (footprint "")
-    )
-    (path "/d7ceb106-986f-4792-af19-7e621a6094bb"
-      (reference "C?") (unit 1) (value "100p") (footprint "")
+      (reference "C5") (unit 1) (value "1n") (footprint "")
+    )
+    (path "/d00eb9ac-8064-45d4-80d1-ec33fd5c15ea"
+      (reference "R1") (unit 1) (value "33k") (footprint "")
     )
     (path "/704d9097-459e-4894-8526-99dda34dca52"
-      (reference "R1") (unit 1) (value "3.3k") (footprint "")
-    )
-    (path "/d00eb9ac-8064-45d4-80d1-ec33fd5c15ea"
-      (reference "R?") (unit 1) (value "33k") (footprint "")
+      (reference "R2") (unit 1) (value "3.3k") (footprint "")
     )
     (path "/c6bb589d-bdf1-405f-a57c-066bfe847b47"
